File: Theremin/Theremin.kicad_sch (KiCad schematic)
At the start: 34 parts, among them J1 9VIN, J2 DIN-5, J3 OUT, J4 MIC, J5 9VOUT, J6 3V3OUT, SW1 SW_Push, SW2 SW_Push, U1 LM317_TO-220, U2 MCP1702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

Commit message: Separate voltage regulators for each oscillator and fix dac output
Parts:
- removed C3: 1u, Capacitor_THT:C_Rect_L7.0mm_W4.5mm_P5.00mm, symbol Device:C_Small
- removed U2: MCP1702, Package_TO_SOT_THT:TO-92_Inline, symbol Regulator_Linear:LM79L12_TO92
- added R6: 240, Resistor_THT:R_Axial_DIN0207_L6.3mm_D2.5mm_P10.16mm_Horizontal, symbol Device:R_Small
- added RV5: 10k, Potentiometer_THT:Potentiometer_Bourns_3299W_Vertical, symbol Device:R_Potentiometer_Small
- added RV8: 10k, Connector_JST:JST_PH_B3B-PH-K_1x03_P2.00mm_Vertical, symbol Device:R_Potentiometer_Small
- added U2: LM317_TO-220, Package_TO_SOT_THT:TO-220-3_Vertical, symbol Regulator_Linear:LM317_TO-220
Connections:
- net +3V3: now also RV8.3
- net +9V: now also U1.3 (VI), U2.3 (VI); no longer C1.1
- net GND: now also RV5.1, RV5.2, RV8.1; no longer U1.3 (VI)
- net NOODLE: now also A1.21 (A2); no longer A1.22 (A3)
- net TONE: now also RV8.2; no longer C2.1
- net +5V renamed V_OSC1
- net V_OSC1: no longer U4.4 (R), U4.8 (VCC)
- new net: R6.2, RV5.3, U2.1 (ADJ)
- new net DAC_OUT: A1.22 (A3), C2.1
- new net V_OSC2: C1.1, R6.1, U2.2 (VO), U4.4 (R), U4.8 (VCC)
- no-connect marks 19 -> 18
Other:
- note removed: "Use optionally instead of MCP1702"
- moved on the sheet: A1, C2, C4, C5, H1, J1, J2, J3, J4, J5, J6, L1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
